File: kicad/punchy.sch (KiCad schematic (older format))
At the start: 22 parts, among them J1 PROG, P1 BATT, Q1 DMG1012T-7, U1 HC05, U2 AP7333, U3 MSP430G2X53, U4 MPU6050

Commit message: Added data dump for dmp, added text to schematic explaining why DMG1012t-7 will not work in its configuration. Can be fixed by flipping source and drain or using p-channel fet
Other:
- note added: "The DMG1012t-7 has an internal diode from source to drain.\nIt also has a gate protection diode \n"
Changed lines of the file:
@@
 Sheet 1 1
 Title "punchy-v1"
-Date "18 jul 2014"
+Date "22 aug 2014"
 Rev "1"
 Comp ""
@@
 Wire Wire Line
 	9650 2050 9650 1850
+Text Notes 700  5850 0    60   ~ 0
+The DMG1012t-7 has an internal diode from source to drain.\nIt also has a gate protection diode \n
 $EndSCHEMATC
